Commit message: base_local_planner working

File: ros/docker/rtabmap/rtabmap_launch/urdf/cuber.urdf (robot description, URDF)
Before this commit: robot cuber, 5 links, 4 joints
Joints:
- joint novatel_center_joint: child novatel_center -> base_link; origin xyz=0 0 0.6858 rpy=0 3.141592653589 0 -> xyz=0 0 0.6858 rpy=0 3.141592653589 3.141592653589; parent base_link -> novatel_center
