Commit message: Add teleop to gazebo Dockerfile and attempt to implement stereo camera in Gazebo

File: ros/docker/gazebo/igvc_self_drive_sim/igvc_self_drive_description/urdf/gem_sensors.urdf.xacro (robot description, xacro)
@@ -7,4 +7,9 @@
     <origin xyz="1.75 0 2.1" rpy="0 0.55 0" />
   </xacro:camera_sim>
+  <!-- Stereo Camera -->
+  <!-- <xacro:include filename="$(find igvc_self_drive_description)/urdf/sensors/stereo.sdf.xacro" />
+  <xacro:camera_sim name="camera_front" parent="base_footprint" >
+    <origin xyz="1.75 0 2.1" rpy="0 0.55 0" />
+  </xacro:camera_sim> -->
   <!-- LIDAR -->
   <xacro:include filename="$(find hector_sensors_description)/urdf/hokuyo_utm30lx.urdf.xacro" />

Commit message: Add stereo camera support in gazebo

File: ros/docker/gazebo/igvc_self_drive_sim/igvc_self_drive_description/urdf/gem_sensors.urdf.xacro (robot description, xacro)
@@ -3,13 +3,13 @@
   <xacro:property name="M_PI" value="3.1415926535897931" />
   <!-- Camera -->
-  <xacro:include filename="$(find igvc_self_drive_description)/urdf/sensors/camera.urdf.xacro" />
-  <xacro:camera_sim name="camera_front" parent="base_footprint" >
-    <origin xyz="1.75 0 2.1" rpy="0 0.55 0" />
-  </xacro:camera_sim>
-  <!-- Stereo Camera -->
-  <!-- <xacro:include filename="$(find igvc_self_drive_description)/urdf/sensors/stereo.sdf.xacro" />
+  <!-- <xacro:include filename="$(find igvc_self_drive_description)/urdf/sensors/camera.urdf.xacro" />
   <xacro:camera_sim name="camera_front" parent="base_footprint" >
     <origin xyz="1.75 0 2.1" rpy="0 0.55 0" />
   </xacro:camera_sim> -->
+  <!-- Stereo Camera -->
+  <xacro:include filename="$(find hector_sensors_description)/urdf/generic_stereo_camera.urdf.xacro" />
+  <xacro:generic_stereo_camera name="stereo_front" parent="base_footprint" ros_topic="sensor_msgs/Image" cam_info_topic="sensor_msgs/CameraInfo" update_rate="30.0" res_x="800" res_y="800" image_format="R8G8B8" hfov="1.396" baseline="0"   >
+    <origin xyz="1.75 0 2.1" rpy="0 0.55 0" />
+  </xacro:generic_stereo_camera>
   <!-- LIDAR -->
   <xacro:include filename="$(find hector_sensors_description)/urdf/hokuyo_utm30lx.urdf.xacro" />

Commit message: Add kinect sensor for gazebo and add bash script to run mapping in gazebo

File: ros/docker/gazebo/igvc_self_drive_sim/igvc_self_drive_description/urdf/gem_sensors.urdf.xacro (robot description, xacro)
@@ -8,8 +8,13 @@
   </xacro:camera_sim> -->
   <!-- Stereo Camera -->
-  <xacro:include filename="$(find hector_sensors_description)/urdf/generic_stereo_camera.urdf.xacro" />
+  <!-- <xacro:include filename="$(find hector_sensors_description)/urdf/generic_stereo_camera.urdf.xacro" />
   <xacro:generic_stereo_camera name="stereo_front" parent="base_footprint" ros_topic="sensor_msgs/Image" cam_info_topic="sensor_msgs/CameraInfo" update_rate="30.0" res_x="800" res_y="800" image_format="R8G8B8" hfov="1.396" baseline="0"   >
     <origin xyz="1.75 0 2.1" rpy="0 0.55 0" />
-  </xacro:generic_stereo_camera>
+  </xacro:generic_stereo_camera> -->
+  <!-- Kinect Camera -->
+  <xacro:include filename="$(find hector_sensors_description)/urdf/kinect_camera.urdf.xacro" />
+  <xacro:kinect_camera name="kinect_camera_model" parent="base_footprint"   >
+    <origin xyz="1.75 0 2.1" rpy="0 0.55 0" />
+  </xacro:kinect_camera>
   <!-- LIDAR -->
   <xacro:include filename="$(find hector_sensors_description)/urdf/hokuyo_utm30lx.urdf.xacro" />
@@ -23,5 +28,5 @@
   </xacro:gps>
   <!-- Sonar sensors -->
-  <xacro:include filename="$(find hector_sensors_description)/urdf/sonar_sensor.urdf.xacro" />
+  <!-- <xacro:include filename="$(find hector_sensors_description)/urdf/sonar_sensor.urdf.xacro" />
   <xacro:sonar_sensor name="front_center" parent="base_footprint" ros_topic="sonar/front_center" update_rate="20" min_range="0.1" max_range="2" field_of_view="0.17" ray_count="3" >
     <origin xyz="2.8 0 0.5" rpy="0 0 0" />
@@ -53,4 +58,4 @@
   <xacro:sonar_sensor name="right_side_rear" parent="base_footprint" ros_topic="sonar/right_side_rear" update_rate="20" min_range="0.1" max_range="2" field_of_view="0.17" ray_count="3" >
     <origin xyz="0 -0.71 0.71" rpy="0 0 ${-M_PI/2}" />
-  </xacro:sonar_sensor>
+  </xacro:sonar_sensor> -->
 </robot>

Commit message: add extra sensors to gazebo, rtabmap_gazebo launch not working yet

File: ros/docker/gazebo/igvc_self_drive_sim/igvc_self_drive_description/urdf/gem_sensors.urdf.xacro (robot description, xacro)
@@ -7,9 +7,24 @@
     <origin xyz="1.75 0 2.1" rpy="0 0.55 0" />
   </xacro:camera_sim> -->
+  <!-- Published Topics -->
+  <!-- /stereo_front/left/camera_info
+       /stereo_front/left/image_raw
+       /stereo_front/left/parameter_descriptions
+       /stereo_front/left/parameter_updates
+       /stereo_front/right/camera_info
+       /stereo_front/right/image_raw
+       /stereo_front/right/parameter_descriptions
+       /stereo_front/right/parameter_updates -->
   <!-- Stereo Camera -->
-  <!-- <xacro:include filename="$(find hector_sensors_description)/urdf/generic_stereo_camera.urdf.xacro" />
+  <xacro:include filename="$(find hector_sensors_description)/urdf/generic_stereo_camera.urdf.xacro" />
   <xacro:generic_stereo_camera name="stereo_front" parent="base_footprint" ros_topic="sensor_msgs/Image" cam_info_topic="sensor_msgs/CameraInfo" update_rate="30.0" res_x="800" res_y="800" image_format="R8G8B8" hfov="1.396" baseline="0"   >
     <origin xyz="1.75 0 2.1" rpy="0 0.55 0" />
-  </xacro:generic_stereo_camera> -->
+  </xacro:generic_stereo_camera>
+  <!-- Published Topics -->
+  <!-- /kinect_camera_model/depth/camera_info
+       /kinect_camera_model/depth/image_raw
+       /kinect_camera_model/depth/points
+       /kinect_camera_model/rgb/camera_info
+       /kinect_camera_model/rgb/image_raw -->
   <!-- Kinect Camera -->
   <xacro:include filename="$(find hector_sensors_description)/urdf/kinect_camera.urdf.xacro" />
@@ -17,4 +32,30 @@
     <origin xyz="1.75 0 2.1" rpy="0 0.55 0" />
   </xacro:kinect_camera>
+  <!-- Published Topics -->
+  <!-- /realsense_camera_model/depth/camera_info
+       /realsense_camera_model/depth/image_raw
+       /realsense_camera_model/depth/points
+       /realsense_camera_model/parameter_descriptions
+       /realsense_camera_model/parameter_updates
+       /realsense_camera_model/rgb/camera_info
+       /realsense_camera_model/rgb/rgb/image_raw -->
+  <!-- Realsense Camera -->
+  <!-- <xacro:include filename="$(find hector_sensors_description)/urdf/realsense_camera.urdf.xacro" />
+  <xacro:realsense_camera name="realsense_camera_model" parent="base_footprint"   >
+    <origin xyz="1.75 0 2.1" rpy="0 0.55 0" />
+  </xacro:realsense_camera> -->
+  <!-- Published Topics -->
+  <!-- /realsense_d435_camera_model/color/camera_info
+       /realsense_d435_camera_model/color/image_raw
+       /realsense_d435_camera_model/depth/camera_info
+       /realsense_d435_camera_model/depth/image_raw
+       /realsense_d435_camera_model/depth/points
+       /realsense_d435_camera_model/parameter_descriptions
+       /realsense_d435_camera_model/parameter_updates -->
+  <!-- Realsense d435 Camera -->
+  <xacro:include filename="$(find hector_sensors_description)/urdf/realsense_d435_camera.urdf.xacro" />
+  <xacro:realsense_d435_camera name="realsense_d435_camera_model" parent="base_footprint"   >
+    <origin xyz="1.75 0 2.1" rpy="0 0.55 0" />
+  </xacro:realsense_d435_camera>
   <!-- LIDAR -->
   <xacro:include filename="$(find hector_sensors_description)/urdf/hokuyo_utm30lx.urdf.xacro" />

Commit message: Bump igvc_self_drive_sim to noetic-devel branch

File: ros/docker/gazebo/igvc_self_drive_sim/igvc_self_drive_description/urdf/gem_sensors.urdf.xacro (robot description, xacro)
@@ -3,59 +3,8 @@
   <xacro:property name="M_PI" value="3.1415926535897931" />
   <!-- Camera -->
-  <!-- <xacro:include filename="$(find igvc_self_drive_description)/urdf/sensors/camera.urdf.xacro" />
+  <xacro:include filename="$(find igvc_self_drive_description)/urdf/sensors/camera.urdf.xacro" />
   <xacro:camera_sim name="camera_front" parent="base_footprint" >
     <origin xyz="1.75 0 2.1" rpy="0 0.55 0" />
-  </xacro:camera_sim> -->
-  <!-- Published Topics -->
-  <!-- /stereo_front/left/camera_info
-       /stereo_front/left/image_raw
-       /stereo_front/left/parameter_descriptions
-       /stereo_front/left/parameter_updates
-       /stereo_front/right/camera_info
-       /stereo_front/right/image_raw
-       /stereo_front/right/parameter_descriptions
-       /stereo_front/right/parameter_updates -->
-  <!-- Stereo Camera -->
-  <xacro:include filename="$(find hector_sensors_description)/urdf/generic_stereo_camera.urdf.xacro" />
-  <xacro:generic_stereo_camera name="stereo_front" parent="base_footprint" ros_topic="sensor_msgs/Image" cam_info_topic="sensor_msgs/CameraInfo" update_rate="30.0" res_x="800" res_y="800" image_format="R8G8B8" hfov="1.396" baseline="0"   >
-    <origin xyz="1.75 0 2.1" rpy="0 0.55 0" />
-  </xacro:generic_stereo_camera>
-  <!-- Published Topics -->
-  <!-- /kinect_camera_model/depth/camera_info
-       /kinect_camera_model/depth/image_raw
-       /kinect_camera_model/depth/points
-       /kinect_camera_model/rgb/camera_info
-       /kinect_camera_model/rgb/image_raw -->
-  <!-- Kinect Camera -->
-  <xacro:include filename="$(find hector_sensors_description)/urdf/kinect_camera.urdf.xacro" />
-  <xacro:kinect_camera name="kinect_camera_model" parent="base_footprint"   >
-    <origin xyz="1.75 0 2.1" rpy="0 0.55 0" />
-  </xacro:kinect_camera>
-  <!-- Published Topics -->
-  <!-- /realsense_camera_model/depth/camera_info
-       /realsense_camera_model/depth/image_raw
-       /realsense_camera_model/depth/points
-       /realsense_camera_model/parameter_descriptions
-       /realsense_camera_model/parameter_updates
-       /realsense_camera_model/rgb/camera_info
-       /realsense_camera_model/rgb/rgb/image_raw -->
-  <!-- Realsense Camera -->
-  <!-- <xacro:include filename="$(find hector_sensors_description)/urdf/realsense_camera.urdf.xacro" />
-  <xacro:realsense_camera name="realsense_camera_model" parent="base_footprint"   >
-    <origin xyz="1.75 0 2.1" rpy="0 0.55 0" />
-  </xacro:realsense_camera> -->
-  <!-- Published Topics -->
-  <!-- /realsense_d435_camera_model/color/camera_info
-       /realsense_d435_camera_model/color/image_raw
-       /realsense_d435_camera_model/depth/camera_info
-       /realsense_d435_camera_model/depth/image_raw
-       /realsense_d435_camera_model/depth/points
-       /realsense_d435_camera_model/parameter_descriptions
-       /realsense_d435_camera_model/parameter_updates -->
-  <!-- Realsense d435 Camera -->
-  <xacro:include filename="$(find hector_sensors_description)/urdf/realsense_d435_camera.urdf.xacro" />
-  <xacro:realsense_d435_camera name="realsense_d435_camera_model" parent="base_footprint"   >
-    <origin xyz="1.75 0 2.1" rpy="0 0.55 0" />
-  </xacro:realsense_d435_camera>
+  </xacro:camera_sim>
   <!-- LIDAR -->
   <xacro:include filename="$(find hector_sensors_description)/urdf/hokuyo_utm30lx.urdf.xacro" />
@@ -69,5 +18,5 @@
   </xacro:gps>
   <!-- Sonar sensors -->
-  <!-- <xacro:include filename="$(find hector_sensors_description)/urdf/sonar_sensor.urdf.xacro" />
+  <xacro:include filename="$(find hector_sensors_description)/urdf/sonar_sensor.urdf.xacro" />
   <xacro:sonar_sensor name="front_center" parent="base_footprint" ros_topic="sonar/front_center" update_rate="20" min_range="0.1" max_range="2" field_of_view="0.17" ray_count="3" >
     <origin xyz="2.8 0 0.5" rpy="0 0 0" />
@@ -99,4 +48,4 @@
   <xacro:sonar_sensor name="right_side_rear" parent="base_footprint" ros_topic="sonar/right_side_rear" update_rate="20" min_range="0.1" max_range="2" field_of_view="0.17" ray_count="3" >
     <origin xyz="0 -0.71 0.71" rpy="0 0 ${-M_PI/2}" />
-  </xacro:sonar_sensor> -->
+  </xacro:sonar_sensor>
 </robot>

Commit message: Remove sonars and add vlp-16

File: ros/docker/gazebo/igvc_self_drive_sim/igvc_self_drive_description/urdf/gem_sensors.urdf.xacro (robot description, xacro)
@@ -17,35 +17,9 @@
     <origin xyz="0.8 0 2.35" rpy="0 0 0" />
   </xacro:gps>
-  <!-- Sonar sensors -->
-  <xacro:include filename="$(find hector_sensors_description)/urdf/sonar_sensor.urdf.xacro" />
-  <xacro:sonar_sensor name="front_center" parent="base_footprint" ros_topic="sonar/front_center" update_rate="20" min_range="0.1" max_range="2" field_of_view="0.17" ray_count="3" >
-    <origin xyz="2.8 0 0.5" rpy="0 0 0" />
-  </xacro:sonar_sensor>
-  <xacro:sonar_sensor name="front_left" parent="base_footprint" ros_topic="sonar/front_left" update_rate="20" min_range="0.1" max_range="2" field_of_view="0.17" ray_count="3" >
-    <origin xyz="2.62 0.4 0.9" rpy="0 0 0" />
-  </xacro:sonar_sensor>
-  <xacro:sonar_sensor name="front_right" parent="base_footprint" ros_topic="sonar/front_right" update_rate="20" min_range="0.1" max_range="2" field_of_view="0.17" ray_count="3" >
-    <origin xyz="2.62 -0.4 0.9" rpy="0 0 0" />
-  </xacro:sonar_sensor>
-  <xacro:sonar_sensor name="left_side_front" parent="base_footprint" ros_topic="sonar/left_side_front" update_rate="20" min_range="0.1" max_range="2" field_of_view="0.17" ray_count="3" >
-    <origin xyz="2.4 0.64 0.9" rpy="0 0 ${M_PI/2}" />
-  </xacro:sonar_sensor>
-  <xacro:sonar_sensor name="right_side_front" parent="base_footprint" ros_topic="sonar/right_side_front" update_rate="20" min_range="0.1" max_range="2" field_of_view="0.17" ray_count="3" >
-    <origin xyz="2.4 -0.64 0.9" rpy="0 0 ${-M_PI/2}" />
-  </xacro:sonar_sensor>
-  <xacro:sonar_sensor name="rear_center" parent="base_footprint" ros_topic="sonar/rear_center" update_rate="20" min_range="0.1" max_range="2" field_of_view="0.17" ray_count="3" >
-    <origin xyz="-0.39 0 0.5" rpy="0 0 ${M_PI}" />
-  </xacro:sonar_sensor>
-  <xacro:sonar_sensor name="rear_left" parent="base_footprint" ros_topic="sonar/rear_left" update_rate="20" min_range="0.1" max_range="2" field_of_view="0.17" ray_count="3" >
-    <origin xyz="-0.39 0.6 0.5" rpy="0 0 ${M_PI}" />
-  </xacro:sonar_sensor>
-  <xacro:sonar_sensor name="rear_right" parent="base_footprint" ros_topic="sonar/rear_right" update_rate="20" min_range="0.1" max_range="2" field_of_view="0.17" ray_count="3" >
-    <origin xyz="-0.39 -0.6 0.5" rpy="0 0 ${M_PI}" />
-  </xacro:sonar_sensor>
-  <xacro:sonar_sensor name="left_side_rear" parent="base_footprint" ros_topic="sonar/left_side_rear" update_rate="20" min_range="0.1" max_range="2" field_of_view="0.17" ray_count="3" >
-    <origin xyz="0 0.71 0.71" rpy="0 0 ${M_PI/2}" />
-  </xacro:sonar_sensor>
-  <xacro:sonar_sensor name="right_side_rear" parent="base_footprint" ros_topic="sonar/right_side_rear" update_rate="20" min_range="0.1" max_range="2" field_of_view="0.17" ray_count="3" >
-    <origin xyz="0 -0.71 0.71" rpy="0 0 ${-M_PI/2}" />
-  </xacro:sonar_sensor>
+  <!-- VLP-16 LiDAR -->
+  <!-- skipped setting organize_cloud and gpu -->
+  <xacro:include filename="$(find velodyne_description)/urdf/VLP-16.urdf.xacro"/>
+  <xacro:VLP-16 parent="base_footprint" name="velodyne" topic="/velodyne_points" hz="10" samples="440">
+    <origin xyz="0.95 0 2.5" rpy="0 0 0" />
+  </xacro:VLP-16>
 </robot>
